Commit message: adding inertial matrices

File: src/balancing_bot/description/balancing_bot.urdf.xacro (robot description, xacro)
@@ -1,4 +1,5 @@
 <?xml version="1.0"?>
 <robot xmlns:xacro="http://www.ros.org/wiki/xacro"  name="robot">
+    <xacro:include filename="inertial_macros.xacro"/> <!-- Include the inertial macros for calculating inertia properties of links. -->
     <!-- materials -->
     <material name="grey">
@@ -35,4 +36,7 @@
             </geometry>
         </collision>
+        <xacro:inertial_box mass="0.2" x=".03" y=".1" z=".12">
+            <origin xyz=".015 .05 .06" rpy="0 0 0"/>
+        </xacro:inertial_box>
     </link>
     <joint name="left_wheel_joint" type="continuous">
@@ -55,4 +59,7 @@
             </geometry>
         </collision>
+        <xacro:inertial_cylinder mass="0.1" length=".025" radius=".025">
+            <origin xyz="0 0 0" rpy="0 0 0"/>
+        </xacro:inertial_cylinder>
     </link>
     <joint name="right_wheel_joint" type="continuous">
@@ -75,4 +82,7 @@
             </geometry>
         </collision>
+        <xacro:inertial_cylinder mass="0.1" length=".025" radius=".025">
+            <origin xyz="0 0 0" rpy="0 0 0"/>
+        </xacro:inertial_cylinder>
     </link>
     <joint name="caster_wheel_joint" type="fixed">
@@ -86,5 +96,5 @@
                 <sphere radius="0.0125" />
             </geometry>
-            <material name="black"/>
+            <material name="blue"/>
         </visual>
         <collision>
@@ -94,4 +104,7 @@
             </geometry>
         </collision>
+        <xacro:inertial_sphere mass="0.05" radius="0.0125">
+            <origin xyz="0 0 0" rpy="0 0 0"/>
+        </xacro:inertial_sphere>
     </link>
 </robot>

Commit message: fix mass

File: src/balancing_bot/description/balancing_bot.urdf.xacro (robot description, xacro)
@@ -37,5 +37,5 @@
         </collision>
         <xacro:inertial_box mass="0.2" x=".03" y=".1" z=".12">
-            <origin xyz=".015 .05 .06" rpy="0 0 0"/>
+            <origin xyz="0 0 -.06" rpy="0 0 0"/>
         </xacro:inertial_box>
     </link>
@@ -96,5 +96,5 @@
                 <sphere radius="0.0125" />
             </geometry>
-            <material name="blue"/>
+            <!-- <material name="blue"/> -->
         </visual>
         <collision>
@@ -108,3 +108,8 @@
         </xacro:inertial_sphere>
     </link>
+    <gazebo reference="caster_wheel_link">
+        <material>Gazebo/White</material>
+        <mu1 value="0.001"/>
+        <mu2 value="0.001"/>
+    </gazebo>
 </robot>

Commit message: differential control

File: src/balancing_bot/description/balancing_bot.urdf.xacro (robot description, xacro)
@@ -2,4 +2,5 @@
 <robot xmlns:xacro="http://www.ros.org/wiki/xacro"  name="robot">
     <xacro:include filename="inertial_macros.xacro"/> <!-- Include the inertial macros for calculating inertia properties of links. -->
+    <xacro:include filename="gazebo_control.xacro"/> <!-- Include the gazebo control macros for controlling the robot in Gazebo. -->
     <!-- materials -->
     <material name="grey">
@@ -16,7 +17,22 @@
     </material>
     <!-- This is a simple balancing bot with a base, two wheels, and a caster wheel. -->
-    <link name="base_link"></link>
-    <joint name="base_to_frame_joint" type="fixed">
+    <link name="base_link">
+        <xacro:inertial_box mass="0.01" x="0.1" y="0.1" z="0.1">
+            <origin xyz="0 0 0" rpy="0 0 0"/>
+        </xacro:inertial_box>
+    </link>
+    <joint name="base_to_base2_joint" type="continuous">
         <parent link="base_link"/>
+        <child link="base2_link"/>
+        <axis xyz="0 1 0"/>
+        <origin rpy="0 0 0" xyz="0 0 0"/>
+    </joint>
+    <link name="base2_link">
+        <xacro:inertial_box mass="0.01" x="0.1" y="0.1" z="0.1">
+            <origin xyz="0 0 0" rpy="0 0 0"/>
+        </xacro:inertial_box>
+    </link>
+    <joint name="base2_to_frame_joint" type="fixed">
+        <parent link="base2_link"/>
         <child link="frame_link"/>
         <origin rpy="0 0 0" xyz="0 0 .105"/>
@@ -36,13 +52,15 @@
             </geometry>
         </collision>
-        <xacro:inertial_box mass="0.2" x=".03" y=".1" z=".12">
+        <xacro:inertial_box mass="0.05" x=".03" y=".1" z=".12">
             <origin xyz="0 0 -.06" rpy="0 0 0"/>
         </xacro:inertial_box>
     </link>
     <joint name="left_wheel_joint" type="continuous">
-        <parent link="base_link"/>
+        <parent link="base2_link"/>
         <child link="left_wheel_link"/>
         <origin xyz="0 0.07 0" rpy="-${pi/2} 0 0"/>
-        <axis xyz="0 0 1"/>
+        <axis xyz="0 0 1">
+            <limit effort="10"/>
+        </axis>
     </joint>
     <link name="left_wheel_link">
@@ -59,13 +77,15 @@
             </geometry>
         </collision>
-        <xacro:inertial_cylinder mass="0.1" length=".025" radius=".025">
+        <xacro:inertial_cylinder mass="0.05" length=".025" radius=".025">
             <origin xyz="0 0 0" rpy="0 0 0"/>
         </xacro:inertial_cylinder>
     </link>
     <joint name="right_wheel_joint" type="continuous">
-        <parent link="base_link"/>
+        <parent link="base2_link"/>
         <child link="right_wheel_link"/>
         <origin xyz="0 -0.07 0" rpy="-${pi/2} 0 0"/>
-        <axis xyz="0 0 1"/>
+        <axis xyz="0 0 1">
+            <limit effort="10"/>
+        </axis>
     </joint>
     <link name="right_wheel_link">
@@ -82,5 +102,5 @@
             </geometry>
         </collision>
-        <xacro:inertial_cylinder mass="0.1" length=".025" radius=".025">
+        <xacro:inertial_cylinder mass="0.05" length=".025" radius=".025">
             <origin xyz="0 0 0" rpy="0 0 0"/>
         </xacro:inertial_cylinder>
@@ -104,5 +124,5 @@
             </geometry>
         </collision>
-        <xacro:inertial_sphere mass="0.05" radius="0.0125">
+        <xacro:inertial_sphere mass="0.1" radius="0.0125">
             <origin xyz="0 0 0" rpy="0 0 0"/>
         </xacro:inertial_sphere>
@@ -113,3 +133,11 @@
         <mu2 value="0.001"/>
     </gazebo>
+    <gazebo reference="left_wheel_link">
+        <mu1 value="0.85"/>
+        <mu2 value="0.85"/>
+    </gazebo>
+    <gazebo reference="right_wheel_link">
+        <mu1 value="0.85"/>
+        <mu2 value="0.85"/>
+    </gazebo>
 </robot>
